Commit message: 11 novembre

File: src/hedgehog_system/urdf/hedgehog_description.urdf (robot description, URDF)
Before this commit: robot hedgehog, 2 links, 1 joints
Links:
- added link imu
Joints:
- added joint base_link_to_imu: type fixed, parent base_link, child imu, origin xyz=0.43 0.09 0.0 rpy=0 0 0
- joint base_link_to_laser: origin xyz=0.0 0.0 0.0 rpy=0 0 0 -> xyz=0.35 0.002 0.0 rpy=0 0 0

Commit message: Bunch of trial and error with odometry

File: src/hedgehog_system/urdf/hedgehog_description.urdf (robot description, URDF)
Before this commit: robot hedgehog, 3 links, 2 joints
Joints:
- joint base_link_to_laser: origin xyz=0.35 0.002 0.0 rpy=0 0 0 -> xyz=0.35 0.002 0.2 rpy=0 0 0
